Commit message: added physical properties so other components can be mounted

File: jackal_description/urdf/accessories/velodyne_mount.urdf.xacro (robot description, xacro)
@@ -9,4 +9,15 @@
         </geometry>
       </visual>
+      <collision>
+        <origin xyz="0 0 -0.28" rpy="0.0 0.0 0.0" />
+        <geometry>
+          <mesh filename="package://jackal_description/meshes/velodyne-bracket.stl" scale="0.01 0.01 0.01"/>
+        </geometry>
+      </collision>
+      <inertial>
+        <mass value="0.100" />
+        <origin xyz="0 0 0" rpy="0 0 0" />
+        <inertia ixx="2.632e-4" ixy="0" ixz="0" iyy="2.632e-4" iyz="0" izz="1.62e-4" />
+      </inertial>
     </link>
     <joint name="velodyne_mount_joint" type="fixed">
