Commit message: changed base_link to base_footprint frame

File: jackal_description/urdf/jackal.urdf.xacro (robot description, xacro)
@@ -74,8 +74,8 @@
     <origin xyz="${-wheelbase/2} ${-track/2} ${wheel_vertical_offset}" rpy="0 0 0" />
   </xacro:wheel>
-  <link name="base_link"></link>
-  <joint name="base_link_joint" type="fixed">
+  <link name="base_footprint"></link>
+  <joint name="base_footprint_joint" type="fixed">
     <origin xyz="0 0 0" rpy="0 0 0" />
-    <parent link="base_link"/>
+    <parent link="base_footprint"/>
     <child link="chassis_link" />
   </joint>

Commit message: parametized tf_prefix

File: jackal_description/urdf/jackal.urdf.xacro (robot description, xacro)
@@ -76,6 +76,12 @@
   <link name="base_footprint"></link>
   <joint name="base_footprint_joint" type="fixed">
+    <origin xyz="0 0 0.0325" rpy="0 0 0" />
+    <parent link="base_footprint"/>
+    <child link="base_link" />
+  </joint>
+  <link name="base_link"></link>
+  <joint name="base_link_joint" type="fixed">
     <origin xyz="0 0 0" rpy="0 0 0" />
-    <parent link="base_footprint"/>
+    <parent link="base_link"/>
     <child link="chassis_link" />
   </joint>
