Commit message: changed from front_laser frame to laser frame

File: jackal_description/urdf/accessories.urdf.xacro (robot description, xacro)
@@ -18,9 +18,9 @@
     <sick_lms1xx_mount prefix="$(optenv JACKAL_LASER_MOUNT front)"
                        topic="$(optenv JACKAL_LASER_TOPIC scan)"/>
-    <joint name="$(optenv JACKAL_LASER_MOUNT front)_laser_mount_joint" type="fixed">
+    <joint name="laser_mount_joint" type="fixed">
       <origin xyz="$(optenv JACKAL_LASER_OFFSET 0 0 0)"
               rpy="$(optenv JACKAL_LASER_RPY 0 0 0)" />
       <parent link="$(optenv JACKAL_LASER_MOUNT front)_mount" />
-      <child link="$(optenv JACKAL_LASER_MOUNT front)_laser_mount" />
+      <child link="laser_mount" />
     </joint>
   </xacro:if>

File: jackal_description/urdf/accessories/sick_lms1xx_mount.urdf.xacro (robot description, xacro)
@@ -28,6 +28,6 @@
   <xacro:include filename="$(find lms1xx)/urdf/sick_lms1xx.urdf.xacro" />
   <xacro:macro name="sick_lms1xx_mount" params="prefix topic">
-    <sick_lms1xx frame="${prefix}_laser" topic="${topic}" />
-    <link name="${prefix}_laser_mount">
+    <sick_lms1xx frame="laser" topic="${topic}" />
+    <link name="laser_mount">
       <visual>
         <origin xyz="0 0 0" rpy="0 0 0" />
@@ -39,11 +39,11 @@
       </visual>
     </link>
-    <joint name="${prefix}_laser_joint" type="fixed">
+    <joint name="laser_joint" type="fixed">
       <!-- This offset is from the base of the bracket to the LIDAR's focal point. -->
       <origin xyz="0 0 0.149" rpy="0 0 0" />
-      <parent link="${prefix}_laser_mount" />
-      <child link="${prefix}_laser" />
+      <parent link="laser_mount" />
+      <child link="laser" />
     </joint>
-    <gazebo reference="${prefix}_laser_mount">
+    <gazebo reference="laser_mount">
       <material>Gazebo/DarkGrey</material>
     </gazebo>

File: jackal_description/urdf/custom_example.urdf (robot description, URDF)
Before this commit: robot None, 0 links, 8 joints
Joints:
- removed joint front_laser_mount_joint
- added joint laser_mount_joint: type fixed, parent front_mount, child laser_mount, origin xyz=0 0 0.002 rpy=0 0 0

Commit message: added kinect

File: jackal_description/urdf/accessories.urdf.xacro (robot description, xacro)
@@ -106,3 +106,21 @@
     </joint>
   </xacro:if>
+  <xacro:if value="$(optenv JACKAL_KINECT 0)">
+  <xacro:include filename="$(find jackal_description)/urdf/accessories/kinect.urdf.xacro" />
+    <jackal_kinect/>
+    <joint name="kinect_mount_joint" type="fixed">
+      <origin xyz="0.1 0 0.05" rpy="0 0 0" />
+      <parent link="front_mount" />
+      <child link="kinect_mount" />
+    </joint>
+  </xacro:if>
+  <xacro:if value="$(optenv JACKAL_KINECT_H 0)">
+  <xacro:include filename="$(find jackal_description)/urdf/accessories/kinect.urdf.xacro" />
+    <jackal_kinect/>
+    <joint name="kinect_mount_joint" type="fixed">
+      <origin xyz="0.028 0 0.23" rpy="0 0 0" />
+      <parent link="front_mount" />
+      <child link="kinect_mount" />
+    </joint>
+  </xacro:if>
 </robot>

Commit message: added velodyne sensor

File: jackal_description/urdf/accessories.urdf.xacro (robot description, xacro)
@@ -124,3 +124,11 @@
     </joint>
   </xacro:if>
+  <xacro:if value="$(optenv JACKAL_VELODYNE 0)">
+    <xacro:include filename="$(find jackal_description)/urdf/accessories/velodyne_mount.urdf.xacro" />
+    <velodyne_mount/>
+    <xacro:include filename="$(find velodyne_description)/urdf/VLP-16.urdf.xacro"/> -->
+    <VLP-16 parent="velodyne_mount" name="velodyne" topic="/velodyne_points" hz="10" samples="1024" gpu="false" lasers="16" max_range="100">
+      <origin xyz="0 0 0" rpy="0 0 0" />
+    </VLP-16>
+  </xacro:if>
 </robot>

Commit message: added pan-tilt module

File: jackal_description/urdf/accessories.urdf.xacro (robot description, xacro)
@@ -132,3 +132,25 @@
     </VLP-16>
   </xacro:if>
+  <xacro:if value="$(optenv JACKAL_PAN_TILT 0)">
+   <xacro:include filename="$(find jackal_description)/urdf/accessories/velodyne_mount.urdf.xacro" />
+    <xacro:include filename="$(find common_sensors)/urdf/sensors/hokuyo_utm30lx.urdf.xacro" />
+    <xacro:include filename="$(find jackal_description)/urdf/accessories/pan_tilt_mount.urdf.xacro" />
+    <velodyne_mount/>
+    <xacro:pan_tilt_mount parent="velodyne_mount">
+        <origin xyz="0.0 0.0 0.0" rpy="0 0 0"/>
+    </xacro:pan_tilt_mount>
+    <xacro:hokuyo_utm30lx
+        name="hokuyo"
+        parent="pan_tilt_mount_link"
+        ros_topic="scan"
+        update_rate="30"
+        ray_count="1040"
+        min_angle="130"
+        max_angle="-130" >
+        <origin xyz="0.0 0.0 0.045" rpy="0 0 0"/>
+    </xacro:hokuyo_utm30lx>
+    <gazebo reference="hokuyo_frame">
+			<material>Gazebo/DarkGrey</material>
+		</gazebo>
+  </xacro:if>
 </robot>

Commit message: lowered down the LIDAR

File: jackal_description/urdf/accessories.urdf.xacro (robot description, xacro)
@@ -19,6 +19,6 @@
                        topic="$(optenv JACKAL_LASER_TOPIC scan)"/>
     <joint name="laser_mount_joint" type="fixed">
-      <origin xyz="$(optenv JACKAL_LASER_OFFSET 0 0 0)"
-              rpy="$(optenv JACKAL_LASER_RPY 0 0 0)" />
+      <origin xyz="$(optenv JACKAL_LASER_OFFSET 0.15 0 -0.03)"
+              rpy="$(optenv JACKAL_LASER_RPY 3.1416 0 0)" />
       <parent link="$(optenv JACKAL_LASER_MOUNT front)_mount" />
       <child link="laser_mount" />

File: jackal_description/urdf/accessories/sick_lms1xx_mount.urdf.xacro (robot description, xacro)
@@ -28,5 +28,5 @@
   <xacro:include filename="$(find lms1xx)/urdf/sick_lms1xx.urdf.xacro" />
   <xacro:macro name="sick_lms1xx_mount" params="prefix topic">
-    <sick_lms1xx frame="laser" topic="${topic}" robot_namespace=""/>
+    <sick_lms1xx frame="laser" topic="${topic}" robot_namespace=""  min_angle="-1.74533" max_angle="1.74533"/>
     <link name="laser_mount">
       <visual>
